File: NanoPi-R4S-RTL8125-retrofit.kicad_pcb (KiCad board)
At the start: 4 copper layers, 21.5 x 13.2 mm, 54 parts, among them J1 Conn_01x01, J10 Conn_01x01, J11 Conn_01x01, J12 Conn_01x01, J13 Conn_01x01, J14 Conn_01x01, J2 Conn_01x01, J3 Conn_01x01, J4 Conn_01x01, J5 Conn_01x01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

Commit message: Finish first layout iteration
Parts:
- added H1: ToolingHole, ToolingHole:ToolingHole_JLCSMT, F.Cu at (113.6, 63.1)
- added H2: ToolingHole, ToolingHole:ToolingHole_JLCSMT, F.Cu at (128.5, 52.8)
- moved TP5 3.67 mm to (113.2, 59.5)
Routing:
- net Net-(U1-EEDO/SPISO/LED2): track 15.8 -> 19.5 mm
- net Net-(U1-CKXTAL2): track 2.34 -> 3.12 mm
- net /REG_EN: track 32.2 -> 31.4 mm
- added copper zone on B.Cu, net GND
Other:
- board text added: "2.5GbE PCIe"
- board text added: "JLCJLCJLCJLC"
- board text added: "RST"
- board text removed: "LED2"
- board text removed: "PERSTB"

Commit message: Finalize initial layout revision
Routing:
- net GND: track 18.9 -> 21.1 mm, vias 27 -> 29
Changed lines of the file:
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@@
     (pad "7" smd rect (at 0.45 -0.475 180) (size 0.25 1.1) (layers "F.Cu" "F.Paste" "F.Mask")
       (net 1 "GND") (pinfunction "GND") (pintype "power_in") (thermal_bridge_angle 45))
+    (model "${KIPRJMOD}/lib/3rdparty/3d/C3151906.x3d"
+      (offset (xyz 0 0 0.5))
+      (scale (xyz 1 1 1))
+      (rotate (xyz 180 0 180))
+    )
   )
   (footprint "Capacitor_SMD:C_0402_1005Metric" (layer "F.Cu")
@@
       (scale (xyz 1 1 1))
       (rotate (xyz 0 0 0))
+    )
+    (model "${KIPRJMOD}/lib/3rdparty/3d/xtal_2016.x3d"
+      (offset (xyz 0 0 0))
+      (scale (xyz 1 1 1))
+      (rotate (xyz 180 0 180))
     )
   )
@@
       (rotate (xyz 0 0 0))
     )
+    (model "${KIPRJMOD}/lib/3rdparty/3d/C3013605.x3d"
+      (offset (xyz 0 0 0))
+      (scale (xyz 1 1 1))
+      (rotate (xyz 180 0 -90))
+    )
   )
   (footprint "Signal_Pad:SignalPad" (layer "F.Cu")
@@
     (effects (font (size 0.9 0.9) (thickness 0.13)) (justify left bottom))
   )
-  (gr_text "LED3" (at 126.1 54.8) (layer "F.SilkS")
+  (gr_text "LED3" (at 125.7 54.75) (layer "F.SilkS")
     (effects (font (size 0.9 0.9) (thickness 0.13)) (justify left bottom))
   )
@@
   (segment (start 130.136827 60.896556) (end 130.646555 60.896556) (width 0.127) (layer "F.Cu") (net 1))
   (segment (start 129.625001 61.400002) (end 129.175 60.950001) (width 0.127) (layer "F.Cu") (net 1))
+  (segment (start 129.799999 57.580001) (end 129.919999 57.580001) (width 0.127) (layer "F.Cu") (net 1))
   (segment (start 120.75 56.175) (end 120.725 56.2) (width 0.127) (layer "F.Cu") (net 1))
   (segment (start 114.45 55.35) (end 114.45 54.175) (width 0.127) (layer "F.Cu") (net 1))
@@
   (segment (start 113.6 60.574999) (end 113.6 60.65) (width 0.127) (layer "F.Cu") (net 1))
   (segment (start 120.75 55.05) (end 120.75 56.175) (width 0.127) (layer "F.Cu") (net 1))
+  (segment (start 129.8 54.950001) (end 129.699999 54.950001) (width 0.127) (layer "F.Cu") (net 1))
   (segment (start 130.775 62.575001) (end 131.425 61.925001) (width 0.25) (layer "F.Cu") (net 1))
   (segment (start 117.5 63.005) (end 117.5 63.525) (width 0.127) (layer "F.Cu") (net 1))
@@
   (segment (start 130.775 62.575001) (end 130.775 61.075001) (width 0.25) (layer "F.Cu") (net 1))
   (segment (start 116.19 54.27833) (end 116.268058 54.356388) (width 0.127) (layer "F.Cu") (net 1))
+  (segment (start 129.919999 57.580001) (end 130.3 57.2) (width 0.127) (layer "F.Cu") (net 1))
+  (segment (start 129.8 54.95) (end 129.45 54.6) (width 0.127) (layer "F.Cu") (net 1))
+  (segment (start 130.775 62.575001) (end 130.1 63.25) (width 0.25) (layer "F.Cu") (net 1))
+  (segment (start 129.8 54.950001) (end 129.8 54.95) (width 0.127) (layer "F.Cu") (net 1))
   (segment (start 124.785 57.915) (end 124.8 57.9) (width 0.127) (layer "F.Cu") (net 1))
   (segment (start 129.65 61.400002) (end 129.625001 61.400002) (width 0.127) (layer "F.Cu") (net 1))
@@
   (segment (start 116.19 53.925) (end 116.19 53.965) (width 0.127) (layer "F.Cu") (net 1))
   (via (at 123.325 55.375) (size 0.45) (drill 0.2) (layers "F.Cu" "B.Cu") (net 1))
-  (via (at 130.85 56.400001) (size 0.45) (drill 0.2) (layers "F.Cu" "B.Cu") (free) (net 1))
+  (via (at 130.3 57.2) (size 0.45) (drill 0.2) (layers "F.Cu" "B.Cu") (net 1))
   (via (at 130.249999 58.000001) (size 0.45) (drill 0.2) (layers "F.Cu" "B.Cu") (free) (net 1))
   (via (at 130.136827 60.896556) (size 0.45) (drill 0.2) (layers "F.Cu" "B.Cu") (net 1))
   (via (at 123.45 60.675) (size 0.45) (drill 0.2) (layers "F.Cu" "B.Cu") (net 1))
-  (via (at 131.9 56.400001) (size 0.45) (drill 0.2) (layers "F.Cu" "B.Cu") (free) (net 1))
   (via (at 124.9 56.7) (size 0.45) (drill 0.2) (layers "F.Cu" "B.Cu") (net 1))
   (via (at 115.201502 57.1) (size 0.45) (drill 0.2) (layers "F.Cu" "B.Cu") (net 1))
@@
   (via (at 119.85 52.6) (size 0.45) (drill 0.2) (layers "F.Cu" "B.Cu") (net 1))
   (via (at 123.875 53.675) (size 0.45) (drill 0.2) (layers "F.Cu" "B.Cu") (net 1))
+  (via (at 129.45 54.6) (size 0.45) (drill 0.2) (layers "F.Cu" "B.Cu") (net 1))
+  (via (at 132.7 56.4) (size 0.45) (drill 0.2) (layers "F.Cu" "B.Cu") (free) (net 1))
   (via (at 129.175 60.950001) (size 0.45) (drill 0.2) (layers "F.Cu" "B.Cu") (net 1))
   (via (at 113.925 60.975) (size 0.45) (drill 0.2) (layers "F.Cu" "B.Cu") (net 1))
@@
   (via (at 122.1 63.525) (size 0.45) (drill 0.2) (layers "F.Cu" "B.Cu") (net 1))
   (via (at 117.5 63.525) (size 0.45) (drill 0.2) (layers "F.Cu" "B.Cu") (net 1))
+  (via (at 130.1 63.25) (size 0.45) (drill 0.2) (layers "F.Cu" "B.Cu") (net 1))
   (via (at 131.525 61.000001) (size 0.45) (drill 0.2) (layers "F.Cu" "B.Cu") (net 1))
   (via (at 124.8 57.9) (size 0.45) (drill 0.2) (layers "F.Cu" "B.Cu") (net 1))
@@
   (segment (start 115.8 63) (end 115.2 62.4) (width 0.127) (layer "B.Cu") (net 42))
   (segment (start 124.3 63) (end 121.5 63) (width 0.127) (layer "B.Cu") (net 42))
+  (segment (start 123.572602 55.85) (end 127 55.85) (width 0.127) (layer "F.Cu") (net 43))
   (segment (start 123.222602 56.2) (end 123.572602 55.85) (width 0.127) (layer "F.Cu") (net 43))
-  (segment (start 127.95 55.85) (end 130.2 53.6) (width 0.127) (layer "F.Cu") (net 43))
-  (segment (start 123.572602 55.85) (end 127.95 55.85) (width 0.127) (layer "F.Cu") (net 43))
+  (segment (start 130.2 53.6) (end 129.25 53.6) (width 0.127) (layer "F.Cu") (net 43))
+  (segment (start 129.25 53.6) (end 127 55.85) (width 0.127) (layer "F.Cu") (net 43))
   (segment (start 122.7 56.2) (end 123.222602 56.2) (width 0.127) (layer "F.Cu") (net 43))
   (zone (net 2) (net_name "Net-(U2-IN)") (layer "F.Cu") (hatch edge 0.5)
@@
         (xy 132.1 58.100001)
         (xy 133.05 58.100001)
-        (xy 133.05 57.150001)
+        (xy 133.05 56)
         (xy 132.15 56.000001)
         (xy 130.85 56.000001)
@@
       )
     )
+  )
+  (zone (net 0) (net_name "") (layers "In1.Cu" "In2.Cu" "B.Cu") (hatch edge 0.5)
+    (connect_pads yes (clearance 0))
+    (min_thickness 0.127) (filled_areas_thickness no)
+    (keepout (tracks allowed) (vias allowed) (pads allowed) (copperpour not_allowed) (footprints allowed))
+    (fill (thermal_gap 0.5) (thermal_bridge_width 0.5))
+    (polygon
+      (pts
+        (xy 130.4 55.2)
+        (xy 132.2 55.2)
+        (xy 132.2 57.4)
+        (xy 130.4 57.4)
+      )
+    )

Commit message: Fix swapped voltage divider on regulator and missing GND on NIC
Parts:
- R1: value 68k -> 120k
- R2: value 120k -> 68k
Changed lines of the file:
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@@
     (descr "Resistor SMD 0402 (1005 Metric), square (rectangular) end terminal, IPC_7351 nominal, (Body size source: IPC-SM-782 page 72, https://www.pcb-3d.com/wordpress/wp-content/uploads/ipc-sm-782a_amendment_1_and_2.pdf), generated with kicad-footprint-generator")
     (tags "resistor")
-    (property "LCSC" "C25750")
+    (property "LCSC" "C36871")
     (property "Sheetfile" "NanoPi-R4S-RTL8125-retrofit.kicad_sch")
     (property "Sheetname" "")
@@
         (effects (font (size 1 1) (thickness 0.15)))
     )
-    (fp_text value "120k" (at 0 1.17 90) (layer "F.Fab")
+    (fp_text value "68k" (at 0 1.17 90) (layer "F.Fab")
         (effects (font (size 1 1) (thickness 0.15)))
     )
@@
     (descr "Resistor SMD 0402 (1005 Metric), square (rectangular) end terminal, IPC_7351 nominal, (Body size source: IPC-SM-782 page 72, https://www.pcb-3d.com/wordpress/wp-content/uploads/ipc-sm-782a_amendment_1_and_2.pdf), generated with kicad-footprint-generator")
     (tags "resistor")
-    (property "LCSC" "C36871")
+    (property "LCSC" "C25750")
     (property "Sheetfile" "NanoPi-R4S-RTL8125-retrofit.kicad_sch")
     (property "Sheetname" "")
@@
         (effects (font (size 1 1) (thickness 0.15)))
     )
-    (fp_text value "68k" (at 0 1.17 90) (layer "F.Fab")
+    (fp_text value "120k" (at 0 1.17 90) (layer "F.Fab")
         (effects (font (size 1 1) (thickness 0.15)))
     )
