File: NanoPi-R4S-RTL8125-retrofit.kicad_sch (KiCad schematic)
At the start: 54 parts, among them J1 Conn_01x01, J10 Conn_01x01, J11 Conn_01x01, J12 Conn_01x01, J13 Conn_01x01, J14 Conn_01x01, J2 Conn_01x01, J3 Conn_01x01, J4 Conn_01x01, J5 Conn_01x01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

Commit message: Finish first layout iteration
Parts:
- added H1, H2: ToolingHole, ToolingHole:ToolingHole_JLCSMT, symbol Mechanical:MountingHole
Changed lines of the file:
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@@
+    )
+  )
+  (symbol (lib_id "Mechanical:MountingHole") (at 15.24 194.31 0) (unit 1)
+    (in_bom no) (on_board yes) (dnp no) (fields_autoplaced)
+    (property "Reference" "H1" (at 17.78 193.0979 0)
+      (effects (font (size 1.27 1.27)) (justify left))
+    )
+    (property "Value" "ToolingHole" (at 17.78 195.5221 0)
+      (effects (font (size 1.27 1.27)) (justify left))
+    )
+    (property "Footprint" "ToolingHole:ToolingHole_JLCSMT" (at 15.24 194.31 0)
+      (effects (font (size 1.27 1.27)) hide)
+    )
+    (property "Datasheet" "~" (at 15.24 194.31 0)
+      (effects (font (size 1.27 1.27)) hide)
+    )
+    (instances
+      (project "NanoPi-R4S-RTL8125-retrofit"
+        (path "/7322593b-e9d4-474f-8b73-ac9576c5ce27"
+          (reference "H1") (unit 1)
+        )
+      )
     )
   )
@@
         )
       )
+    )
+  )
+  (symbol (lib_id "Mechanical:MountingHole") (at 15.24 189.23 0) (unit 1)
+    (in_bom no) (on_board yes) (dnp no) (fields_autoplaced)
+    (property "Reference" "H2" (at 17.78 188.0179 0)
+      (effects (font (size 1.27 1.27)) (justify left))
+    )
+    (property "Value" "ToolingHole" (at 17.78 190.4421 0)
+      (effects (font (size 1.27 1.27)) (justify left))
+    )
+    (property "Footprint" "ToolingHole:ToolingHole_JLCSMT" (at 15.24 189.23 0)
+      (effects (font (size 1.27 1.27)) hide)
+    )
+    (property "Datasheet" "~" (at 15.24 189.23 0)
+      (effects (font (size 1.27 1.27)) hide)
+    )
+    (instances
+      (project "NanoPi-R4S-RTL8125-retrofit"
+        (path "/7322593b-e9d4-474f-8b73-ac9576c5ce27"
+          (reference "H2") (unit 1)
+        )
+      )

Commit message: Fix swapped voltage divider on regulator and missing GND on NIC
Parts:
- R1: value 68k -> 120k; LCSC C36871 -> C25750
- R2: value 120k -> 68k; LCSC C25750 -> C36871
Changed lines of the file:
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@@
+    )
+  )
+  (symbol (lib_id "power:GND") (at 143.51 133.35 0) (unit 1)
+    (in_bom yes) (on_board yes) (dnp no) (fields_autoplaced)
+    (property "Reference" "#PWR022" (at 143.51 139.7 0)
+      (effects (font (size 1.27 1.27)) hide)
+    )
+    (property "Value" "GND" (at 143.51 137.4831 0)
+      (effects (font (size 1.27 1.27)))
+    )
+    (property "Footprint" "" (at 143.51 133.35 0)
+      (effects (font (size 1.27 1.27)) hide)
+    )
+    (property "Datasheet" "" (at 143.51 133.35 0)
+      (effects (font (size 1.27 1.27)) hide)
+    )
+    (pin "1")
+    (instances
+      (project "NanoPi-R4S-RTL8125-retrofit"
+        (path "/7322593b-e9d4-474f-8b73-ac9576c5ce27"
+          (reference "#PWR022") (unit 1)
+        )
+      )
     )
   )
@@
       (effects (font (size 1.27 1.27)) (justify left))
     )
-    (property "Value" "120k" (at 124.6886 30.4221 0)
+    (property "Value" "68k" (at 124.6886 30.4221 0)
       (effects (font (size 1.27 1.27)) (justify left))
     )
@@
       (effects (font (size 1.27 1.27)) hide)
     )
-    (property "LCSC" "C25750" (at 123.19 29.21 0)
+    (property "LCSC" "C36871" (at 123.19 29.21 0)
       (effects (font (size 1.27 1.27)) hide)
     )
@@
       (effects (font (size 1.27 1.27)) (justify left))
     )
-    (property "Value" "68k" (at 124.6886 38.0421 0)
+    (property "Value" "120k" (at 124.6886 38.0421 0)
       (effects (font (size 1.27 1.27)) (justify left))
     )
@@
       (effects (font (size 1.27 1.27)) hide)
     )
-    (property "LCSC" "C36871" (at 123.19 36.83 0)
+    (property "LCSC" "C25750" (at 123.19 36.83 0)
       (effects (font (size 1.27 1.27)) hide)
     )
